Commit message: xacro: wire ROS namespace into gz_ros2_control plugin
The plugin hosts controller_manager inside gz, but needs to know which
namespace to look in for robot_description. Added 'ns' xacro arg passed
alongside 'prefix', injected as <ros><namespace>${ns}</namespace></ros>
inside the gz plugin block.

spawn_robot.launch.py now passes ns:=<name> when rendering xacro.

File: brickbot_ws/src/brickbot_description/urdf/brickbot.ros2_control.xacro (robot description, xacro)
@@ -5,5 +5,5 @@
 -->
 <robot xmlns:xacro="http://www.ros.org/wiki/xacro">
-  <xacro:macro name="brickbot_ros2_control" params="prefix">
+  <xacro:macro name="brickbot_ros2_control" params="prefix ns">
     <ros2_control name="${prefix}gz_system" type="system">
       <hardware>
@@ -45,4 +45,7 @@
       <plugin filename="gz_ros2_control-system" name="gz_ros2_control::GazeboSimROS2ControlPlugin">
         <parameters>$(find brickbot_control)/config/controllers.yaml</parameters>
+        <ros>
+          <namespace>${ns}</namespace>
+        </ros>
       </plugin>
     </gazebo>

File: brickbot_ws/src/brickbot_description/urdf/brickbot.urdf.xacro (robot description, xacro)
@@ -8,6 +8,8 @@
   <xacro:arg name="prefix" default=""/>
   <xacro:arg name="tool"   default="gripper"/>
+  <xacro:arg name="ns"     default=""/>
   <xacro:property name="pfx" value="$(arg prefix)"/>
   <xacro:property name="tool_type" value="$(arg tool)"/>
+  <xacro:property name="ns" value="$(arg ns)"/>
   <xacro:include filename="$(find brickbot_description)/urdf/base_tracked.xacro"/>
   <xacro:include filename="$(find brickbot_description)/urdf/arm_6dof.xacro"/>
@@ -25,4 +27,4 @@
     <xacro:tool_cement prefix="${pfx}arm_" parent="${pfx}arm_tool0"/>
   </xacro:if>
-  <xacro:brickbot_ros2_control prefix="${pfx}"/>
+  <xacro:brickbot_ros2_control prefix="${pfx}" ns="${ns}"/>
 </robot>
