Commit message: WIP: backup before laptop repair

File: vika_ws/src/vika_description/urdf/arm_6dof.xacro (robot description, xacro)
@@ -1,10 +1,18 @@
 <?xml version="1.0"?>
 <!--
-  6-DOF serial anthropomorphic arm (RRR-RRR).
-  Per-link STL drop-in: pass mesh_<linkname>:=<package://...> to override the
-  primitive geometry. Empty string keeps the primitive box/cylinder fallback.
+  6-DOF serial arm — mountable on the tracked base.
+  Joint origins are auto-generated by MCP from the Fusion 360 assembly
+  (home pose = current CAD pose), identical to base_only.urdf.xacro:
+    - Every joint origin carries the proximal-joint position AND the rpy that
+      orients the child link's frame.
+    - Every joint axis is therefore the child's local +Z.
+    - The STL meshes are authored AT each joint frame, so every visual/collision
+      origin is identity (0 0 0).
+  Per-link STL drop-in: pass mesh_<linkname>:=<package://...> to override.
+  An EMPTY string falls back to a primitive block placed at the joint frame.
 -->
 <robot xmlns:xacro="http://www.ros.org/wiki/xacro">
   <xacro:macro name="arm_6dof" params="prefix parent
+                                       define_materials:=true
                                        mesh_base_link:='package://vika_description/meshes/arm/ROD-STL/base.stl'
                                        mesh_link1:='package://vika_description/meshes/arm/ROD-STL/link1.stl'
@@ -24,5 +32,9 @@
       </xacro:unless>
     </xacro:macro>
-    <!-- Shoulder mount plate -->
+    <xacro:if value="${define_materials}">
+      <material name="arm_grey"><color rgba="0.3 0.3 0.3 1"/></material>
+      <material name="arm_orange"><color rgba="0.92 0.45 0.10 1"/></material>
+    </xacro:if>
+    <!-- Shoulder mount plate (caller supplies the origin on the base) -->
     <joint name="${prefix}mount_joint" type="fixed">
       <xacro:insert_block name="origin"/>
@@ -32,12 +44,12 @@
     <link name="${prefix}base_link">
       <visual>
-        <origin xyz="0 0 0.075"/>
+        <origin xyz="0 0 0" rpy="0 0 0"/>
         <xacro:geom_or_mesh mesh_uri="${mesh_base_link}">
           <geometry><cylinder radius="0.12" length="0.15"/></geometry>
         </xacro:geom_or_mesh>
-        <material name="arm_grey"><color rgba="0.3 0.3 0.3 1"/></material>
-      </visual>
-      <collision>
-        <origin xyz="0 0 0.075"/>
+        <material name="arm_grey"/>
+      </visual>
+      <collision>
+        <origin xyz="0 0 0" rpy="0 0 0"/>
         <xacro:geom_or_mesh mesh_uri="${mesh_base_link}">
           <geometry><cylinder radius="0.12" length="0.15"/></geometry>
@@ -45,45 +57,45 @@
       </collision>
       <inertial>
-        <mass value="4.0"/>
-        <inertia ixx="0.02" iyy="0.02" izz="0.03" ixy="0" ixz="0" iyz="0"/>
+        <mass value="3.0"/>
+        <inertia ixx="0.05" iyy="0.05" izz="0.08" ixy="0" ixz="0" iyz="0"/>
       </inertial>
     </link>
-    <!-- J1: Base rotation -->
+    <!-- J1: base yaw -->
     <joint name="${prefix}j1" type="revolute">
       <parent link="${prefix}base_link"/>
       <child link="${prefix}link1"/>
-      <origin xyz="0 0 0.15" rpy="0 0 0"/>
-      <axis xyz="0 0 1"/>
-      <limit lower="-3.23" upper="3.23" effort="80" velocity="3.14"/>
+      <origin xyz="0 0 0.175" rpy="0 0 1.5152"/>
+      <axis xyz="0 0 1"/>
+      <limit lower="-3.14" upper="3.14" effort="80" velocity="3.14"/>
       <dynamics damping="0.5" friction="0.1"/>
     </joint>
     <link name="${prefix}link1">
       <visual>
-        <origin xyz="0 0 0.125"/>
+        <origin xyz="0 0 0" rpy="0 0 0"/>
         <xacro:geom_or_mesh mesh_uri="${mesh_link1}">
           <geometry><box size="0.18 0.18 0.25"/></geometry>
         </xacro:geom_or_mesh>
-        <material name="arm_orange"><color rgba="0.9 0.5 0.1 1"/></material>
-      </visual>
-      <collision>
-        <origin xyz="0 0 0.125"/>
+        <material name="arm_orange"/>
+      </visual>
+      <collision>
+        <origin xyz="0 0 0" rpy="0 0 0"/>
         <xacro:geom_or_mesh mesh_uri="${mesh_link1}">
           <geometry><box size="0.18 0.18 0.25"/></geometry>
         </xacro:geom_or_mesh>
       </collision>
-      <inertial><mass value="6.0"/><inertia ixx="0.05" iyy="0.05" izz="0.03" ixy="0" ixz="0" iyz="0"/></inertial>
-    </link>
-    <!-- J2: Shoulder pitch -->
+      <inertial><mass value="6.0"/><inertia ixx="0.10" iyy="0.10" izz="0.06" ixy="0" ixz="0" iyz="0"/></inertial>
+    </link>
+    <!-- J2: shoulder pitch -->
     <joint name="${prefix}j2" type="revolute">
       <parent link="${prefix}link1"/>
       <child link="${prefix}link2"/>
-      <origin xyz="0.1 0 0.25" rpy="0 0 0"/>
-      <axis xyz="0 1 0"/>
-      <limit lower="-2.70" upper="0.61" effort="80" velocity="2.5"/>
+      <origin xyz="0.1038 -0.4023 0.2912" rpy="1.5708 0 -1.5708"/>
+      <axis xyz="0 0 1"/>
+      <limit lower="-2.70" upper="2.70" effort="80" velocity="2.5"/>
       <dynamics damping="0.5" friction="0.1"/>
     </joint>
     <link name="${prefix}link2">
       <visual>
-        <origin xyz="0 0 0.275"/>
+        <origin xyz="0 0 0" rpy="0 0 0"/>
         <xacro:geom_or_mesh mesh_uri="${mesh_link2}">
           <geometry><box size="0.12 0.14 0.55"/></geometry>
@@ -92,23 +104,23 @@
       </visual>
       <collision>
-        <origin xyz="0 0 0.275"/>
+        <origin xyz="0 0 0" rpy="0 0 0"/>
         <xacro:geom_or_mesh mesh_uri="${mesh_link2}">
           <geometry><box size="0.12 0.14 0.55"/></geometry>
         </xacro:geom_or_mesh>
       </collision>
-      <inertial><mass value="5.0"/><inertia ixx="0.14" iyy="0.14" izz="0.02" ixy="0" ixz="0" iyz="0"/></inertial>
-    </link>
-    <!-- J3: Elbow -->
+      <inertial><mass value="5.0"/><inertia ixx="0.7" iyy="0.05" izz="0.7" ixy="0" ixz="0" iyz="0"/></inertial>
+    </link>
+    <!-- J3: elbow -->
     <joint name="${prefix}j3" type="revolute">
       <parent link="${prefix}link2"/>
       <child link="${prefix}link3"/>
-      <origin xyz="0 0 0.55" rpy="0 0 0"/>
-      <axis xyz="0 1 0"/>
-      <limit lower="-2.27" upper="2.69" effort="60" velocity="2.8"/>
+      <origin xyz="0 1.300 0" rpy="0 0 -0.2221"/>
+      <axis xyz="0 0 1"/>
+      <limit lower="-2.70" upper="2.70" effort="60" velocity="2.8"/>
       <dynamics damping="0.5" friction="0.1"/>
     </joint>
     <link name="${prefix}link3">
       <visual>
-        <origin xyz="0 0 0.225"/>
+        <origin xyz="0 0 0" rpy="0 0 0"/>
         <xacro:geom_or_mesh mesh_uri="${mesh_link3}">
           <geometry><box size="0.10 0.12 0.45"/></geometry>
@@ -117,5 +129,5 @@
       </visual>
       <collision>
-        <origin xyz="0 0 0.225"/>
+        <origin xyz="0 0 0" rpy="0 0 0"/>
         <xacro:geom_or_mesh mesh_uri="${mesh_link3}">
           <geometry><box size="0.10 0.12 0.45"/></geometry>
@@ -124,9 +136,9 @@
       <inertial><mass value="3.5"/><inertia ixx="0.07" iyy="0.07" izz="0.01" ixy="0" ixz="0" iyz="0"/></inertial>
     </link>
-    <!-- J4: Wrist roll -->
+    <!-- J4: wrist roll -->
     <joint name="${prefix}j4" type="revolute">
       <parent link="${prefix}link3"/>
       <child link="${prefix}link4"/>
-      <origin xyz="0 0 0.45" rpy="0 0 0"/>
+      <origin xyz="0.1600 0.2369 0.0003" rpy="1.5708 0.9923 1.5708"/>
       <axis xyz="0 0 1"/>
       <limit lower="-6.10" upper="6.10" effort="20" velocity="5.0"/>
@@ -135,5 +147,5 @@
     <link name="${prefix}link4">
       <visual>
-        <origin xyz="0 0 0.06"/>
+        <origin xyz="0 0 0" rpy="0 0 0"/>
         <xacro:geom_or_mesh mesh_uri="${mesh_link4}">
           <geometry><cylinder radius="0.05" length="0.12"/></geometry>
@@ -142,17 +154,17 @@
       </visual>
       <collision>
-        <origin xyz="0 0 0.06"/>
+        <origin xyz="0 0 0" rpy="0 0 0"/>
         <xacro:geom_or_mesh mesh_uri="${mesh_link4}">
           <geometry><cylinder radius="0.05" length="0.12"/></geometry>
         </xacro:geom_or_mesh>
       </collision>
-      <inertial><mass value="1.2"/><inertia ixx="0.002" iyy="0.002" izz="0.001" ixy="0" ixz="0" iyz="0"/></inertial>
-    </link>
-    <!-- J5: Wrist pitch -->
+      <inertial><mass value="1.5"/><inertia ixx="0.05" iyy="0.05" izz="0.005" ixy="0" ixz="0" iyz="0"/></inertial>
+    </link>
+    <!-- J5: wrist pitch -->
     <joint name="${prefix}j5" type="revolute">
       <parent link="${prefix}link4"/>
       <child link="${prefix}link5"/>
-      <origin xyz="0 0 0.12" rpy="0 0 0"/>
-      <axis xyz="0 1 0"/>
+      <origin xyz="-0.0860 0 1.3050" rpy="1.5708 -1.3556 -1.5708"/>
+      <axis xyz="0 0 1"/>
       <limit lower="-2.27" upper="2.27" effort="20" velocity="5.0"/>
       <dynamics damping="0.2" friction="0.05"/>
@@ -160,5 +172,5 @@
     <link name="${prefix}link5">
       <visual>
-        <origin xyz="0 0 0.04"/>
+        <origin xyz="0 0 0" rpy="0 0 0"/>
         <xacro:geom_or_mesh mesh_uri="${mesh_link5}">
           <geometry><box size="0.08 0.08 0.08"/></geometry>
@@ -167,5 +179,5 @@
       </visual>
       <collision>
-        <origin xyz="0 0 0.04"/>
+        <origin xyz="0 0 0" rpy="0 0 0"/>
         <xacro:geom_or_mesh mesh_uri="${mesh_link5}">
           <geometry><box size="0.08 0.08 0.08"/></geometry>
@@ -174,9 +186,9 @@
       <inertial><mass value="0.8"/><inertia ixx="0.001" iyy="0.001" izz="0.001" ixy="0" ixz="0" iyz="0"/></inertial>
     </link>
-    <!-- J6: Tool rotation -->
+    <!-- J6: tool roll. Child carries link6.stl and serves as the tool0 flange. -->
     <joint name="${prefix}j6" type="revolute">
       <parent link="${prefix}link5"/>
       <child link="${prefix}tool0"/>
-      <origin xyz="0 0 0.08" rpy="0 0 0"/>
+      <origin xyz="0.1600 0 -0.0850" rpy="-1.5708 1.3440 -1.5708"/>
       <axis xyz="0 0 1"/>
       <limit lower="-6.10" upper="6.10" effort="15" velocity="6.0"/>
@@ -185,5 +197,5 @@
     <link name="${prefix}tool0">
       <visual>
-        <origin xyz="0 0 0.02"/>
+        <origin xyz="0 0 0" rpy="0 0 0"/>
         <xacro:geom_or_mesh mesh_uri="${mesh_tool0}">
           <geometry><cylinder radius="0.035" length="0.04"/></geometry>
@@ -192,5 +204,5 @@
       </visual>
       <collision>
-        <origin xyz="0 0 0.02"/>
+        <origin xyz="0 0 0" rpy="0 0 0"/>
         <xacro:geom_or_mesh mesh_uri="${mesh_tool0}">
           <geometry><cylinder radius="0.035" length="0.04"/></geometry>

File: vika_ws/src/vika_description/urdf/vika.urdf.xacro (robot description, xacro)
@@ -10,8 +10,12 @@
   <xacro:arg name="ns"     default=""/>
   <xacro:arg name="arm"    default="false"/>
+  <!-- use_meshes:=true loads the Fusion CAD STLs; false uses the primitive
+       box/cylinder fallbacks that match the joint kinematics exactly. -->
+  <xacro:arg name="use_meshes" default="true"/>
   <xacro:property name="pfx" value="$(arg prefix)"/>
   <xacro:property name="tool_type" value="$(arg tool)"/>
   <xacro:property name="ns" value="$(arg ns)"/>
   <xacro:property name="arm_enabled" value="$(arg arm)"/>
+  <xacro:property name="use_meshes" value="$(arg use_meshes)"/>
   <xacro:include filename="$(find vika_description)/urdf/base_tracked.xacro"/>
   <xacro:include filename="$(find vika_description)/urdf/arm_6dof.xacro"/>
@@ -21,7 +25,16 @@
   <xacro:base_tracked prefix="${pfx}"/>
   <xacro:if value="${arm_enabled}">
-    <xacro:arm_6dof prefix="${pfx}arm_" parent="${pfx}base_link">
-      <origin xyz="-0.3 0 0.2" rpy="0 0 0"/>
-    </xacro:arm_6dof>
+    <xacro:if value="${use_meshes}">
+      <xacro:arm_6dof prefix="${pfx}arm_" parent="${pfx}base_link">
+        <origin xyz="-0.3 0 0.2" rpy="0 0 0"/>
+      </xacro:arm_6dof>
+    </xacro:if>
+    <xacro:unless value="${use_meshes}">
+      <xacro:arm_6dof prefix="${pfx}arm_" parent="${pfx}base_link"
+                      mesh_base_link="" mesh_link1="" mesh_link2="" mesh_link3=""
+                      mesh_link4="" mesh_link5="" mesh_tool0="">
+        <origin xyz="-0.3 0 0.2" rpy="0 0 0"/>
+      </xacro:arm_6dof>
+    </xacro:unless>
     <xacro:if value="${tool_type == 'gripper'}">
       <xacro:tool_gripper prefix="${pfx}arm_" parent="${pfx}arm_tool0"/>
