Commit message: WIP: stable 3x3 respawn masonry (single dynamic pick-row)
Replace the fragile 36-brick 3x4 pallet (tall stacks toppled on reset/pick)
with a single dynamic pick-row row_0_0 that respawns after each course:
- construction_site.sdf: one flat row on the pallet (was 12 fused rows)
- tool_gripper.xacro: one DetachableJoint /suction/r0_0 (was 12)
- bridge.yaml: one suction attach/detach pair (was 24)
- lay_course.sh / reset_bricks.sh: spawn 3 static wall bricks + teleport
  row_0_0 back to the pallet
- bt_node.py _build: 3-wide x 3-high wall, one pick-row per course
- start-docker.sh stop_sim: also kill bt_node/hmi_bridge/dino/move_group so
  restarts don't leave stale duplicate nodes running pre-edit code

File: vika_ws/src/vika_description/urdf/arm_6dof.xacro (robot description, xacro)
@@ -33,6 +33,6 @@
     </xacro:macro>
     <xacro:if value="${define_materials}">
-      <material name="arm_grey"><color rgba="0.3 0.3 0.3 1"/></material>
-      <material name="arm_orange"><color rgba="0.92 0.45 0.10 1"/></material>
+      <material name="arm_grey"><color rgba="0.16 0.16 0.18 1"/></material>
+      <material name="arm_orange"><color rgba="0.95 0.45 0.10 1"/></material>
     </xacro:if>
     <!-- Shoulder mount plate (caller supplies the origin on the base) -->
@@ -52,7 +52,6 @@
       <collision>
         <origin xyz="0 0 0" rpy="0 0 0"/>
-        <xacro:geom_or_mesh mesh_uri="${mesh_base_link}">
-          <geometry><cylinder radius="0.12" length="0.15"/></geometry>
-        </xacro:geom_or_mesh>
+        <!-- primitive collision (cheap) — mesh kept for visual only -->
+        <geometry><cylinder radius="0.12" length="0.15"/></geometry>
       </collision>
       <inertial>
@@ -67,5 +66,5 @@
       <origin xyz="0 0 0.175" rpy="0 0 1.5152"/>
       <axis xyz="0 0 1"/>
-      <limit lower="-3.14" upper="3.14" effort="80" velocity="3.14"/>
+      <limit lower="-3.14" upper="3.14" effort="800" velocity="3.14"/>
       <dynamics damping="0.5" friction="0.1"/>
     </joint>
@@ -76,11 +75,9 @@
           <geometry><box size="0.18 0.18 0.25"/></geometry>
         </xacro:geom_or_mesh>
-        <material name="arm_orange"/>
-      </visual>
-      <collision>
-        <origin xyz="0 0 0" rpy="0 0 0"/>
-        <xacro:geom_or_mesh mesh_uri="${mesh_link1}">
-          <geometry><box size="0.18 0.18 0.25"/></geometry>
-        </xacro:geom_or_mesh>
+        <material name="arm_grey"/>
+      </visual>
+      <collision>
+        <origin xyz="0 0 0" rpy="0 0 0"/>
+        <geometry><box size="0.18 0.18 0.25"/></geometry>
       </collision>
       <inertial><mass value="6.0"/><inertia ixx="0.10" iyy="0.10" izz="0.06" ixy="0" ixz="0" iyz="0"/></inertial>
@@ -92,5 +89,5 @@
       <origin xyz="0.1038 -0.4023 0.2912" rpy="1.5708 0 -1.5708"/>
       <axis xyz="0 0 1"/>
-      <limit lower="-2.70" upper="2.70" effort="80" velocity="2.5"/>
+      <limit lower="-2.70" upper="2.70" effort="800" velocity="2.5"/>
       <dynamics damping="0.5" friction="0.1"/>
     </joint>
@@ -101,11 +98,9 @@
           <geometry><box size="0.12 0.14 0.55"/></geometry>
         </xacro:geom_or_mesh>
-        <material name="arm_orange"/>
-      </visual>
-      <collision>
-        <origin xyz="0 0 0" rpy="0 0 0"/>
-        <xacro:geom_or_mesh mesh_uri="${mesh_link2}">
-          <geometry><box size="0.12 0.14 0.55"/></geometry>
-        </xacro:geom_or_mesh>
+        <material name="arm_grey"/>
+      </visual>
+      <collision>
+        <origin xyz="0 0 0" rpy="0 0 0"/>
+        <geometry><box size="0.12 0.14 0.55"/></geometry>
       </collision>
       <inertial><mass value="5.0"/><inertia ixx="0.7" iyy="0.05" izz="0.7" ixy="0" ixz="0" iyz="0"/></inertial>
@@ -117,5 +112,5 @@
       <origin xyz="0 1.300 0" rpy="0 0 -0.2221"/>
       <axis xyz="0 0 1"/>
-      <limit lower="-2.70" upper="2.70" effort="60" velocity="2.8"/>
+      <limit lower="-2.70" upper="2.70" effort="500" velocity="2.8"/>
       <dynamics damping="0.5" friction="0.1"/>
     </joint>
@@ -126,11 +121,9 @@
           <geometry><box size="0.10 0.12 0.45"/></geometry>
         </xacro:geom_or_mesh>
-        <material name="arm_orange"/>
-      </visual>
-      <collision>
-        <origin xyz="0 0 0" rpy="0 0 0"/>
-        <xacro:geom_or_mesh mesh_uri="${mesh_link3}">
-          <geometry><box size="0.10 0.12 0.45"/></geometry>
-        </xacro:geom_or_mesh>
+        <material name="arm_grey"/>
+      </visual>
+      <collision>
+        <origin xyz="0 0 0" rpy="0 0 0"/>
+        <geometry><box size="0.10 0.12 0.45"/></geometry>
       </collision>
       <inertial><mass value="3.5"/><inertia ixx="0.07" iyy="0.07" izz="0.01" ixy="0" ixz="0" iyz="0"/></inertial>
@@ -142,5 +135,5 @@
       <origin xyz="0.1600 0.2369 0.0003" rpy="1.5708 0.9923 1.5708"/>
       <axis xyz="0 0 1"/>
-      <limit lower="-6.10" upper="6.10" effort="20" velocity="5.0"/>
+      <limit lower="-6.10" upper="6.10" effort="300" velocity="5.0"/>
       <dynamics damping="0.2" friction="0.05"/>
     </joint>
@@ -155,7 +148,5 @@
       <collision>
         <origin xyz="0 0 0" rpy="0 0 0"/>
-        <xacro:geom_or_mesh mesh_uri="${mesh_link4}">
-          <geometry><cylinder radius="0.05" length="0.12"/></geometry>
-        </xacro:geom_or_mesh>
+        <geometry><cylinder radius="0.05" length="0.12"/></geometry>
       </collision>
       <inertial><mass value="1.5"/><inertia ixx="0.05" iyy="0.05" izz="0.005" ixy="0" ixz="0" iyz="0"/></inertial>
@@ -167,5 +158,5 @@
       <origin xyz="-0.0860 0 1.3050" rpy="1.5708 -1.3556 -1.5708"/>
       <axis xyz="0 0 1"/>
-      <limit lower="-2.27" upper="2.27" effort="20" velocity="5.0"/>
+      <limit lower="-2.27" upper="2.27" effort="300" velocity="5.0"/>
       <dynamics damping="0.2" friction="0.05"/>
     </joint>
@@ -180,7 +171,5 @@
       <collision>
         <origin xyz="0 0 0" rpy="0 0 0"/>
-        <xacro:geom_or_mesh mesh_uri="${mesh_link5}">
-          <geometry><box size="0.08 0.08 0.08"/></geometry>
-        </xacro:geom_or_mesh>
+        <geometry><box size="0.08 0.08 0.08"/></geometry>
       </collision>
       <inertial><mass value="0.8"/><inertia ixx="0.001" iyy="0.001" izz="0.001" ixy="0" ixz="0" iyz="0"/></inertial>
@@ -192,5 +181,5 @@
       <origin xyz="0.1600 0 -0.0850" rpy="-1.5708 1.3440 -1.5708"/>
       <axis xyz="0 0 1"/>
-      <limit lower="-6.10" upper="6.10" effort="15" velocity="6.0"/>
+      <limit lower="-6.10" upper="6.10" effort="150" velocity="6.0"/>
       <dynamics damping="0.1" friction="0.02"/>
     </joint>
@@ -205,7 +194,5 @@
       <collision>
         <origin xyz="0 0 0" rpy="0 0 0"/>
-        <xacro:geom_or_mesh mesh_uri="${mesh_tool0}">
-          <geometry><cylinder radius="0.035" length="0.04"/></geometry>
-        </xacro:geom_or_mesh>
+        <geometry><cylinder radius="0.035" length="0.04"/></geometry>
       </collision>
       <inertial><mass value="0.3"/><inertia ixx="0.0002" iyy="0.0002" izz="0.0002" ixy="0" ixz="0" iyz="0"/></inertial>

File: vika_ws/src/vika_description/urdf/tool_cement.xacro (robot description, xacro)
@@ -31,4 +31,31 @@
     </joint>
     <link name="${prefix}tcp"/>
+    <!-- Wrist camera on the cement tool: looks down the tool +Z at the laid wall
+         (DINO cement-following). Mirrors the gripper wrist cam. Distinct gz topic
+         (${prefix}wrist_cam) so it doesn't clash with robot_a's /wrist_cam. -->
+    <joint name="${prefix}wrist_cam_joint" type="fixed">
+      <parent link="${prefix}cement_base"/>
+      <child link="${prefix}wrist_cam_link"/>
+      <origin xyz="0.12 0 0.05" rpy="0 -1.5708 0"/>
+    </joint>
+    <link name="${prefix}wrist_cam_link">
+      <visual><geometry><box size="0.03 0.03 0.03"/></geometry></visual>
+      <inertial><mass value="0.05"/><inertia ixx="1e-5" iyy="1e-5" izz="1e-5" ixy="0" ixz="0" iyz="0"/></inertial>
+    </link>
+    <gazebo reference="${prefix}wrist_cam_link">
+      <sensor name="wrist_cam" type="camera">
+        <pose>0 0 0 0 0 0</pose>
+        <always_on>1</always_on>
+        <update_rate>15</update_rate>
+        <visualize>true</visualize>
+        <topic>${prefix}wrist_cam</topic>
+        <gz_frame_id>${prefix}wrist_cam_link</gz_frame_id>
+        <camera>
+          <horizontal_fov>1.3</horizontal_fov>
+          <image><width>640</width><height>480</height><format>R8G8B8</format></image>
+          <clip><near>0.02</near><far>10.0</far></clip>
+        </camera>
+      </sensor>
+    </gazebo>
   </xacro:macro>
 </robot>

File: vika_ws/src/vika_description/urdf/tool_gripper.xacro (robot description, xacro)
@@ -1,64 +1,113 @@
 <?xml version="1.0"?>
-<!-- Parallel-jaw gripper with mimic joint. -->
+<!-- Vacuum suction gripper sized to pick THREE bricks at once.
+     A wide mounting bar (gripper_base) + 3 round suction pads, one per brick
+     (bricks are 0.375 x 0.25 m, picked side-by-side along the bar's Y axis).
+     Picking is on/off suction, so there are NO actuated joints. The link name
+     `gripper_base` is kept because MoveIt (vika.srdf) and build_wall.py attach
+     carried bricks to it; `tcp` is the suction contact frame (centre pad). -->
 <robot xmlns:xacro="http://www.ros.org/wiki/xacro">
-  <xacro:macro name="tool_gripper" params="prefix parent
-                                           mesh_gripper:='package://vika_description/meshes/arm/ROD-STL/gripper.stl'">
+  <xacro:macro name="tool_gripper" params="prefix parent">
+    <material name="tool_grey"><color rgba="0.4 0.4 0.45 1"/></material>
+    <material name="suction_black"><color rgba="0.12 0.12 0.14 1"/></material>
+    <!-- Wide mounting bar on the wrist flange (spans 3 bricks along Y) -->
     <joint name="${prefix}gripper_base_joint" type="fixed">
       <parent link="${parent}"/>
       <child link="${prefix}gripper_base"/>
-      <origin xyz="0 0 0.04"/>
+      <origin xyz="0 0 0.02"/>
     </joint>
     <link name="${prefix}gripper_base">
       <visual>
-        <xacro:if value="${len(mesh_gripper) &gt; 0}">
-          <geometry><mesh filename="${mesh_gripper}" scale="0.001 0.001 0.001"/></geometry>
-        </xacro:if>
-        <xacro:unless value="${len(mesh_gripper) &gt; 0}">
-          <geometry><box size="0.10 0.08 0.05"/></geometry>
-        </xacro:unless>
-        <material name="tool_grey"><color rgba="0.4 0.4 0.45 1"/></material>
+        <origin xyz="0 0 0.02"/>
+        <!-- bar spans the 3 pads at y=±0.375 (+pad radius) — 0.95 m is plenty;
+             the old 1.45 m was sized for the wider 0.5 m pad spacing. -->
+        <geometry><box size="0.34 0.95 0.04"/></geometry>
+        <material name="tool_grey"/>
       </visual>
-      <collision>
-        <xacro:if value="${len(mesh_gripper) &gt; 0}">
-          <geometry><mesh filename="${mesh_gripper}" scale="0.001 0.001 0.001"/></geometry>
-        </xacro:if>
-        <xacro:unless value="${len(mesh_gripper) &gt; 0}">
-          <geometry><box size="0.10 0.08 0.05"/></geometry>
-        </xacro:unless>
-      </collision>
-      <inertial><mass value="0.5"/><inertia ixx="0.0005" iyy="0.0005" izz="0.0005" ixy="0" ixz="0" iyz="0"/></inertial>
+      <!-- No collision geometry: grasping is via the DetachableJoint (not contact),
+           and the long bar's collision caused false self-collisions with the base
+           that blocked motion / MoveIt planning. -->
+      <inertial><mass value="1.2"/><inertia ixx="0.07" iyy="0.02" izz="0.08" ixy="0" ixz="0" iyz="0"/></inertial>
     </link>
-    <joint name="${prefix}gripper_left_finger" type="prismatic">
-      <parent link="${prefix}gripper_base"/>
-      <child link="${prefix}left_finger"/>
-      <origin xyz="0 0.02 0.05"/>
-      <axis xyz="0 1 0"/>
-      <limit lower="0.0" upper="0.04" effort="60" velocity="0.1"/>
-    </joint>
-    <link name="${prefix}left_finger">
-      <visual><geometry><box size="0.02 0.015 0.08"/></geometry><origin xyz="0 0 0.04"/><material name="tool_grey"/></visual>
-      <collision><geometry><box size="0.02 0.015 0.08"/></geometry><origin xyz="0 0 0.04"/></collision>
-      <inertial><mass value="0.1"/><inertia ixx="0.0001" iyy="0.0001" izz="0.0001" ixy="0" ixz="0" iyz="0"/></inertial>
-    </link>
-    <joint name="${prefix}gripper_right_finger" type="prismatic">
-      <parent link="${prefix}gripper_base"/>
-      <child link="${prefix}right_finger"/>
-      <origin xyz="0 -0.02 0.05"/>
-      <axis xyz="0 -1 0"/>
-      <limit lower="0.0" upper="0.04" effort="60" velocity="0.1"/>
-      <mimic joint="${prefix}gripper_left_finger" multiplier="1.0" offset="0"/>
-    </joint>
-    <link name="${prefix}right_finger">
-      <visual><geometry><box size="0.02 0.015 0.08"/></geometry><origin xyz="0 0 0.04"/><material name="tool_grey"/></visual>
-      <collision><geometry><box size="0.02 0.015 0.08"/></geometry><origin xyz="0 0 0.04"/></collision>
-      <inertial><mass value="0.1"/><inertia ixx="0.0001" iyy="0.0001" izz="0.0001" ixy="0" ixz="0" iyz="0"/></inertial>
-    </link>
-    <!-- TCP frame -->
+    <!-- One suction pad per brick, centred at the three brick positions (Y) -->
+    <xacro:macro name="suction_pad" params="name y">
+      <joint name="${prefix}${name}_joint" type="fixed">
+        <parent link="${prefix}gripper_base"/>
+        <child link="${prefix}${name}"/>
+        <origin xyz="0 ${y} 0.06"/>
+      </joint>
+      <link name="${prefix}${name}">
+        <visual>
+          <geometry><cylinder radius="0.09" length="0.04"/></geometry>
+          <material name="suction_black"/>
+        </visual>
+        <!-- no collision (attach-based grasping) -->
+        <inertial><mass value="0.15"/><inertia ixx="0.0002" iyy="0.0002" izz="0.0003" ixy="0" ixz="0" iyz="0"/></inertial>
+      </link>
+    </xacro:macro>
+    <!-- pad spacing 0.375 = brick long side EXACTLY, so the placed row sits
+         flush (zero gap) along world X. With the längs pick yaw the bar (local
+         Y) runs along world X = along the bricks' long axis. -->
+    <xacro:suction_pad name="suction_pad_l" y="0.375"/>
+    <xacro:suction_pad name="suction_pad_c" y="0.0"/>
+    <xacro:suction_pad name="suction_pad_r" y="-0.375"/>
+    <!-- TCP at the centre pad contact face -->
     <joint name="${prefix}tcp_joint" type="fixed">
-      <parent link="${prefix}gripper_base"/>
+      <parent link="${prefix}suction_pad_c"/>
       <child link="${prefix}tcp"/>
-      <origin xyz="0 0 0.13"/>
+      <origin xyz="0 0 0.02"/>
     </joint>
     <link name="${prefix}tcp"/>
+    <!-- Wrist camera: mounted at the bar edge (clear of the pads), looking down
+         the tool +Z (= world -Z when the gripper is top-down) at the bricks.
+         gz cameras look along the sensor frame +X, so pitch -90deg aims +X at
+         the parent +Z. Used by the DINO brick detector + HMI wrist view. -->
+    <joint name="${prefix}wrist_cam_joint" type="fixed">
+      <parent link="${prefix}gripper_base"/>
+      <child link="${prefix}wrist_cam_link"/>
+      <origin xyz="0.22 0 0.03" rpy="0 -1.5708 0"/>
+    </joint>
+    <link name="${prefix}wrist_cam_link">
+      <visual>
+        <geometry><box size="0.03 0.03 0.03"/></geometry>
+        <material name="suction_black"/>
+      </visual>
+      <inertial><mass value="0.05"/><inertia ixx="1e-5" iyy="1e-5" izz="1e-5" ixy="0" ixz="0" iyz="0"/></inertial>
+    </link>
+    <gazebo reference="${prefix}wrist_cam_link">
+      <sensor name="wrist_cam" type="camera">
+        <pose>0 0 0 0 0 0</pose>
+        <always_on>1</always_on>
+        <update_rate>15</update_rate>
+        <visualize>true</visualize>
+        <topic>wrist_cam</topic>
+        <gz_frame_id>${prefix}wrist_cam_link</gz_frame_id>
+        <camera>
+          <horizontal_fov>1.3</horizontal_fov>
+          <image><width>640</width><height>480</height><format>R8G8B8</format></image>
+          <clip><near>0.02</near><far>10.0</far></clip>
+        </camera>
+      </sensor>
+    </gazebo>
+    <!-- Vacuum "suction": one gz DetachableJoint per brick. Each starts DETACHED
+         (attach_topic given) and creates a fixed joint to its brick model when
+         an Empty msg hits the attach topic; the detach topic releases it.
+         NOTE: the suction-pad links are lumped into ${prefix}tool0 by URDF->SDF
+         fixed-joint reduction, so the surviving parent link is tool0. The brick
+         attaches at its current relative pose, so it stays under its pad. -->
+    <!-- ONE DetachableJoint for the single dynamic pick-ROW (3 fused bricks, model
+         row_0_0). The gripper grabs the whole row; after laying a course as STATIC
+         wall bricks the row is teleported back to the pallet (respawn build). The
+         flat single row never topples (unlike the old 3x4 pallet stack). -->
+    <gazebo>
+      <plugin filename="gz-sim-detachable-joint-system" name="gz::sim::systems::DetachableJoint">
+        <parent_link>${prefix}tool0</parent_link>
+        <child_model>row_0_0</child_model>
+        <child_link>row</child_link>
+        <attach_topic>/suction/r0_0/attach</attach_topic>
+        <detach_topic>/suction/r0_0/detach</detach_topic>
+        <output_topic>/suction/r0_0/state</output_topic>
+        <suppress_child_warning>true</suppress_child_warning>
+      </plugin>
+    </gazebo>
   </xacro:macro>
 </robot>

File: vika_ws/src/vika_description/urdf/vika.ros2_control.xacro (robot description, xacro)
@@ -10,30 +10,32 @@
         <plugin>gz_ros2_control/GazeboSimSystem</plugin>
       </hardware>
-      <!-- Base drive is handled by native gz DiffDrive plugin, not ros2_control. -->
-      <!-- Arm joints are controlled through ros2_control / MoveIt. -->
-      <!-- Arm -->
-      <xacro:macro name="arm_joint_ifc" params="name">
+      <!-- Linear rail carriage (prismatic, world +Y). Held + commandable. -->
+      <joint name="${prefix}rail_joint">
+        <command_interface name="position"/>
+        <state_interface name="position">
+          <param name="initial_value">0.0</param>
+        </state_interface>
+        <state_interface name="velocity"/>
+      </joint>
+      <!-- Arm. initial_value = a folded "stow" pose so the robots spawn compact
+           instead of both reaching toward the centre and overlapping ("kissing").
+           Matches the FOLD pose the startup script commands the controllers to. -->
+      <xacro:macro name="arm_joint_ifc" params="name init:=0.0">
         <joint name="${name}">
           <command_interface name="position"/>
           <state_interface name="position">
-            <param name="initial_value">0.0</param>
+            <param name="initial_value">${init}</param>
           </state_interface>
           <state_interface name="velocity"/>
         </joint>
       </xacro:macro>
-      <xacro:arm_joint_ifc name="${prefix}arm_j1"/>
-      <xacro:arm_joint_ifc name="${prefix}arm_j2"/>
-      <xacro:arm_joint_ifc name="${prefix}arm_j3"/>
-      <xacro:arm_joint_ifc name="${prefix}arm_j4"/>
-      <xacro:arm_joint_ifc name="${prefix}arm_j5"/>
-      <xacro:arm_joint_ifc name="${prefix}arm_j6"/>
-      <!-- Gripper (only left finger has a command; right mimics via URDF) -->
-      <xacro:if value="${tool == 'gripper'}">
-        <joint name="${prefix}arm_gripper_left_finger">
-          <command_interface name="position"/>
-          <state_interface name="position"/>
-          <state_interface name="velocity"/>
-        </joint>
-      </xacro:if>
+      <xacro:arm_joint_ifc name="${prefix}arm_j1" init="1.5708"/>
+      <xacro:arm_joint_ifc name="${prefix}arm_j2" init="0.0"/>
+      <xacro:arm_joint_ifc name="${prefix}arm_j3" init="0.6"/>
+      <xacro:arm_joint_ifc name="${prefix}arm_j4" init="0.0"/>
+      <xacro:arm_joint_ifc name="${prefix}arm_j5" init="0.0"/>
+      <xacro:arm_joint_ifc name="${prefix}arm_j6" init="0.0"/>
+      <!-- Vacuum suction gripper has no actuated joint (on/off suction), so it
+           contributes no ros2_control interfaces. -->
       <!-- Cement nozzle angle -->
       <xacro:if value="${tool == 'cement'}">

File: vika_ws/src/vika_description/urdf/vika.urdf.xacro (robot description, xacro)
@@ -10,4 +10,8 @@
   <xacro:arg name="ns"     default=""/>
   <xacro:arg name="arm"    default="false"/>
+  <!-- World anchor for this robot (spawn pose is ignored by the world-fixed
+       rail, so bake placement here). base_yaw=3.14159 faces the robot -X. -->
+  <xacro:arg name="base_x"   default="0"/>
+  <xacro:arg name="base_yaw" default="0"/>
   <!-- use_meshes:=true loads the Fusion CAD STLs; false uses the primitive
        box/cylinder fallbacks that match the joint kinematics exactly. -->
@@ -17,15 +21,18 @@
   <xacro:property name="ns" value="$(arg ns)"/>
   <xacro:property name="arm_enabled" value="$(arg arm)"/>
+  <xacro:property name="base_x" value="$(arg base_x)"/>
+  <xacro:property name="base_yaw" value="$(arg base_yaw)"/>
   <xacro:property name="use_meshes" value="$(arg use_meshes)"/>
-  <xacro:include filename="$(find vika_description)/urdf/base_tracked.xacro"/>
+  <xacro:include filename="$(find vika_description)/urdf/base_rail.xacro"/>
   <xacro:include filename="$(find vika_description)/urdf/arm_6dof.xacro"/>
   <xacro:include filename="$(find vika_description)/urdf/tool_gripper.xacro"/>
   <xacro:include filename="$(find vika_description)/urdf/tool_cement.xacro"/>
   <xacro:include filename="$(find vika_description)/urdf/vika.ros2_control.xacro"/>
-  <xacro:base_tracked prefix="${pfx}"/>
+  <!-- Linear rail base: arm rides a prismatic carriage along world +Y. -->
+  <xacro:base_rail prefix="${pfx}" base_x="${base_x}" base_yaw="${base_yaw}"/>
   <xacro:if value="${arm_enabled}">
     <xacro:if value="${use_meshes}">
       <xacro:arm_6dof prefix="${pfx}arm_" parent="${pfx}base_link">
-        <origin xyz="-0.3 0 0.2" rpy="0 0 0"/>
+        <origin xyz="0 0 0.09" rpy="0 0 0"/>
       </xacro:arm_6dof>
     </xacro:if>
@@ -34,5 +41,5 @@
                       mesh_base_link="" mesh_link1="" mesh_link2="" mesh_link3=""
                       mesh_link4="" mesh_link5="" mesh_tool0="">
-        <origin xyz="-0.3 0 0.2" rpy="0 0 0"/>
+        <origin xyz="0 0 0.09" rpy="0 0 0"/>
       </xacro:arm_6dof>
     </xacro:unless>
@@ -45,8 +52,10 @@
   </xacro:if>
   <!--
-    ros2_control integration disabled for Phase 2.
-    Base driving uses the native gz DiffDrive system plugin (see base_tracked.xacro).
-    Arm control will be re-enabled together with MoveIt2 in a later phase.
+    ros2_control + gz_ros2_control: actuates the rail + arm (+ tool) joints so
+    they hold position under gravity. Without this the unactuated revolute
+    joints sag and the robot "collapses". Requires arm:=true.
   -->
-  <!-- <xacro:vika_ros2_control prefix="${pfx}" ns="${ns}" tool="${tool_type}"/> -->
+  <xacro:if value="${arm_enabled}">
+    <xacro:vika_ros2_control prefix="${pfx}" ns="${ns}" tool="${tool_type}"/>
+  </xacro:if>
 </robot>
