Commit message: WIP: working 3x3 build + cement demo (single-row respawn, top-down place, J4 unlock)
VIKA-6 builds a 3-long x 3-high running-bond wall and VIKA-5 cements between
courses — full demo runs end-to-end, web-triggered (HMI BUILD -> rosbridge -> bt).

Brick build:
- pallet = 1 dynamic respawning pick-row (row_0_0) + 2 STATIC deco rows (reliable
  pick; the 3-dynamic-rows respawn was flaky)
- TOP-DOWN placement: hover high over the x/y target, then descend straight down in
  Z (Cartesian MoveL) -> sets the row from above, no sideways snag on neighbours
- lay_course.sh whisk-first (dynamic row away, then spawn static) -> no overlap
  explosion; wall_brick.sdf keeps collision so rows rest

Cement (VIKA-5) — the hard part:
- IK tip is cement_BASE (per SRDF), so target it at a reachable height; the long-ish
  nozzle puts the TIP down at the bricks
- **J4 unlock** (vika.urdf.xacro lock_j4=false): the zero-range [0,0] J4 lock made
  MoveIt CheckStartStateBounds reject every cement plan (START_STATE_INVALID) so
  VIKA-5 never moved. Unlocking it (the older working config) fixed it.
- HOME_POSE j1 1.5708 -> 1.55 (was exactly at the limit -> same rejection)

Ops:
- restart-clean.sh: reliable one-command restart (full docker restart purges DDS
  ghosts + the controller spawner lock-race; retries until controllers active)
- start-docker.sh stop_sim also kills bt_node/hmi_bridge/dino/move_group

Known polish TODO: wrist-cam renders dark (headless EGL fails on NVIDIA/Wayland);
VIKA-6 J6 wrist-roll spins more than necessary between längs pick and yawed place.

File: vika_ws/src/vika_description/urdf/arm_6dof.xacro (robot description, xacro)
@@ -15,4 +15,5 @@
   <xacro:macro name="arm_6dof" params="prefix parent
                                        define_materials:=true
+                                       lock_j4:=false
                                        mesh_base_link:='package://vika_description/meshes/arm/ROD-STL/base.stl'
                                        mesh_link1:='package://vika_description/meshes/arm/ROD-STL/link1.stl'
@@ -135,5 +136,17 @@
       <origin xyz="0.1600 0.2369 0.0003" rpy="1.5708 0.9923 1.5708"/>
       <axis xyz="0 0 1"/>
-      <limit lower="-6.10" upper="6.10" effort="300" velocity="5.0"/>
+      <!-- lock_j4 (VIKA-5 / cement): wrist-roll about the rotationally-symmetric
+           nozzle is functionless, so the doc'd 5-DOF arm HARD-locks it to 0
+           (zero-range limit -> the joint cannot move, realising 5 DOF). -->
+      <xacro:if value="${lock_j4}">
+        <!-- NOT a zero range [0,0]: the joint never reports EXACTLY 0 (float noise
+             ~1e-13), so [0,0] makes MoveIt's CheckStartStateBounds reject every plan
+             that STARTS there ("Start state out of bounds") — that silently blocked
+             VIKA-5's cement IK. A tiny ±0.05 range keeps it effectively 5-DOF/locked. -->
+        <limit lower="-0.05" upper="0.05" effort="300" velocity="5.0"/>
+      </xacro:if>
+      <xacro:unless value="${lock_j4}">
+        <limit lower="-6.10" upper="6.10" effort="300" velocity="5.0"/>
+      </xacro:unless>
       <dynamics damping="0.2" friction="0.05"/>
     </joint>

File: vika_ws/src/vika_description/urdf/base_rail.xacro (robot description, xacro)
@@ -53,6 +53,8 @@
       <origin xyz="0 0 0.15" rpy="0 0 0"/>
       <axis xyz="0 1 0"/>
-      <limit lower="${(lay_sign-1)*travel/2}" upper="${(lay_sign+1)*travel/2}" effort="2000" velocity="0.8"/>
-      <dynamics damping="50.0" friction="20.0"/>
+      <limit lower="${(lay_sign-1)*travel/2}" upper="${(lay_sign+1)*travel/2}" effort="4000" velocity="3.0"/>
+      <!-- low damping/no static friction: the old 50/20 stalled the position-PID so
+           the carriage never actually slid (controller reported reached, joint frozen). -->
+      <dynamics damping="2.0" friction="0.0"/>
     </joint>
     <!-- Carriage: a dark slider centred on the rail, footprint matching the arm
@@ -65,8 +67,6 @@
         <material name="carriage_dark"/>
       </visual>
-      <collision>
-        <origin xyz="0 0 0.0" rpy="0 0 0"/>
-        <geometry><box size="0.9 0.9 0.18"/></geometry>
-      </collision>
+      <!-- no collision: the carriage is kinematically held by the prismatic joint;
+           a collision box only risks jamming the slide against the rail/ground. -->
       <inertial>
         <mass value="40.0"/>

File: vika_ws/src/vika_description/urdf/tool_cement.xacro (robot description, xacro)
@@ -20,7 +20,12 @@
       <limit lower="-1.57" upper="1.57" effort="5" velocity="1.0"/>
     </joint>
+    <!-- LONG thin nozzle: the tip (tcp) sits 0.33 m below the angle joint (0.45 m
+         below the wrist). VIKA-5 then holds its WRIST at the comfortably-reachable
+         height while the long nozzle reaches all the way DOWN to the brick top — so
+         the tip applies cement AT the bricks without the arm contorting at full
+         stretch. No collision on the nozzle (thin cosmetic tool; collision would make
+         the planner avoid the wall it's meant to touch). -->
     <link name="${prefix}nozzle">
-      <visual><geometry><cylinder radius="0.015" length="0.08"/></geometry><origin xyz="0 0 0.04"/><material name="tool_red"/></visual>
-      <collision><geometry><cylinder radius="0.015" length="0.08"/></geometry><origin xyz="0 0 0.04"/></collision>
+      <visual><geometry><cylinder radius="0.015" length="0.23"/></geometry><origin xyz="0 0 0.115"/><material name="tool_red"/></visual>
       <inertial><mass value="0.1"/><inertia ixx="0.0001" iyy="0.0001" izz="0.0001" ixy="0" ixz="0" iyz="0"/></inertial>
     </link>
@@ -28,5 +33,5 @@
       <parent link="${prefix}nozzle"/>
       <child link="${prefix}tcp"/>
-      <origin xyz="0 0 0.08"/>
+      <origin xyz="0 0 0.23"/>
     </joint>
     <link name="${prefix}tcp"/>

File: vika_ws/src/vika_description/urdf/vika.urdf.xacro (robot description, xacro)
@@ -32,11 +32,16 @@
   <xacro:base_rail prefix="${pfx}" base_x="${base_x}" base_yaw="${base_yaw}"/>
   <xacro:if value="${arm_enabled}">
+    <!-- J4 (wrist-roll) is left FREE. It was hard-locked for VIKA-5 (cement) to claim
+         a 5-DOF arm, but the zero-range lock made MoveIt reject every cement plan
+         ("Start state out of bounds") so VIKA-5 never moved to cement. Unlocked = the
+         working configuration; wrist-roll is harmless (the nozzle is symmetric). -->
+    <xacro:property name="lock_j4" value="false"/>
     <xacro:if value="${use_meshes}">
-      <xacro:arm_6dof prefix="${pfx}arm_" parent="${pfx}base_link">
+      <xacro:arm_6dof prefix="${pfx}arm_" parent="${pfx}base_link" lock_j4="${lock_j4}">
         <origin xyz="0 0 0.09" rpy="0 0 0"/>
       </xacro:arm_6dof>
     </xacro:if>
     <xacro:unless value="${use_meshes}">
-      <xacro:arm_6dof prefix="${pfx}arm_" parent="${pfx}base_link"
+      <xacro:arm_6dof prefix="${pfx}arm_" parent="${pfx}base_link" lock_j4="${lock_j4}"
                       mesh_base_link="" mesh_link1="" mesh_link2="" mesh_link3=""
                       mesh_link4="" mesh_link5="" mesh_tool0="">
